File: Head Tracking FPV/Receiver/Receiver PCB/Receiver PCB.kicad_sch (KiCad schematic)
At the start: 7 parts, among them J1 Conn_01x02_Pin, J2 Pan Servo, J3 Tilt Servo, J4 Conn_01x05_Pin, J5 VTX Power, SW1 SW_SPDT, U1 ESP32-DEVKIT-V1

Commit message: Added Mounting Holes
Parts:
- added H1, H2, H3, H4: MountingHole, MountingHole:MountingHole_3.2mm_M3, symbol Mechanical:MountingHole
